File: pcb/BattleBot.kicad_pcb (KiCad board)
At the start: 4 copper layers, 109.5 x 58.5 mm, 20 parts, among them J1 WeaponMotor, J2 Motor1, J3 Motor2

Commit message: polish
Parts:
- Receiver1: footprint BattleBot:Reciever -> BattleBot:Receiver
Changed lines of the file:
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@@
 		(embedded_fonts no)
 	)
-	(footprint "BattleBot:Reciever"
+	(footprint "BattleBot:Receiver"
 		(layer "F.Cu")
 		(at 199.8 82.636628 -90)
