File: pcb/BattleBot.kicad_sch (KiCad schematic)
At the start: 19 parts, among them J1 WeaponMotor, J2 Motor1, J3 Motor2

Commit message: polish
Parts:
- Receiver1: footprint BattleBot:Reciever -> BattleBot:Receiver
Changed lines of the file:
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@@
 			)
 		)
-		(property "Footprint" "BattleBot:Reciever"
+		(property "Footprint" "BattleBot:Receiver"
 			(at 20.32 130.81 0)
 			(hide yes)
